File: Driver Board.brd (EAGLE design)
At the start: 100 x 80 mm, 25 parts, among them Q1 IRF7389, Q2 IRF7389, Q5 IRF7389, X1 5566-8, X2 5566-8

Commit message: im a muthafucking commit
Parts:
- removed Q3, Q4, Q6: (no value), semicon-smd-ipc:SOT23
- added T1, T2, T3: (no value), zetex:SOT223
- moved R13 93.6 mm to (48.3, 20.3)
- moved R15 93.6 mm to (38.1, 20.3)
- moved R5 92.6 mm to (41.9, 2.54)
- moved R4 86.9 mm to (43.2, 7.62), turned to 90 degrees
- moved R6 82.4 mm to (33.0, 20.3), turned to 180 degrees
- moved R7 81.1 mm to (26.7, 20.3), turned to 180 degrees
- moved R3 77.5 mm to (43.2, 20.3)
- moved R8 74.5 mm to (53.3, 20.3)
- moved R14 73.0 mm to (16.5, 11.4), turned to 90 degrees
- moved R12 64.2 mm to (21.6, 20.3)
- moved R11 55.3 mm to (16.5, 20.3)
- moved R1 43.4 mm to (14.0, 17.8)
- moved C1 26.9 mm to (55.9, 7.62), turned to 90 degrees
- moved Q5 12.0 mm to (20.3, 16.5)
- moved R9 11.4 mm to (24.1, 2.54)
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Connections:
- net GND: now also T1.3, T2.3, T3.3; no longer Q3.2, Q4.2, Q6.2
- net N$1: now also T1.2; no longer Q3.3
- net N$11: now also T3.2; no longer Q6.3
- net N$13: now also T3.1; no longer Q6.1
- net N$2: now also T2.2; no longer Q4.3
- net N$5: now also T1.1; no longer Q3.1
- net N$6: now also T2.1; no longer Q4.1
Other:
- outline, holes or cut-outs redrawn
