File: Driver Board.sch (EAGLE design)
At the start: 25 parts, among them Q1 IRF7389, Q2 IRF7389, Q5 IRF7389, X1 5566-8, X2 5566-8

Commit message: im a muthafucking commit
Parts:
- removed Q3, Q4, Q6: (no value), semicon-smd-ipc:NPN-TRANSISTOR_SOT23
- added T1, T2, T3: (no value), zetex:NPNSOT223
Connections:
- net GND: now also T1.E, T2.E, T3.E; no longer Q3.E, Q4.E, Q6.E
- net N$1: now also T1.C1; no longer Q3.C
- net N$11: now also T3.C1; no longer Q6.C
- net N$13: now also T3.B; no longer Q6.B
- net N$2: now also T2.C1; no longer Q4.C
- net N$5: now also T1.B; no longer Q3.B
- net N$6: now also T2.B; no longer Q4.B
Changed lines of the file:
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@@
 <part name="U$1" library="ATmega48" deviceset="ATMEGA48" device=""/>
 <part name="Q1" library="transistor-fet" deviceset="IRF7389" device=""/>
-<part name="Q3" library="semicon-smd-ipc" deviceset="NPN-TRANSISTOR_" device="SOT23"/>
 <part name="R1" library="rcl" deviceset="R-US_" device="R1206"/>
 <part name="R2" library="rcl" deviceset="R-US_" device="R1206"/>
@@
 <part name="R5" library="rcl" deviceset="R-US_" device="R1206"/>
 <part name="Q2" library="transistor-fet" deviceset="IRF7389" device=""/>
-<part name="Q4" library="semicon-smd-ipc" deviceset="NPN-TRANSISTOR_" device="SOT23"/>
 <part name="R6" library="rcl" deviceset="R-US_" device="R1206"/>
 <part name="R7" library="rcl" deviceset="R-US_" device="R1206"/>
@@
 <part name="R10" library="rcl" deviceset="R-US_" device="R1206"/>
 <part name="Q5" library="transistor-fet" deviceset="IRF7389" device=""/>
-<part name="Q6" library="semicon-smd-ipc" deviceset="NPN-TRANSISTOR_" device="SOT23"/>
 <part name="R11" library="rcl" deviceset="R-US_" device="R1206"/>
 <part name="R12" library="rcl" deviceset="R-US_" device="R1206"/>
@@
 <part name="X2" library="con-molex" deviceset="5566-8" device=""/>
 <part name="C1" library="resistor" deviceset="C-US" device="C1206"/>
+<part name="T1" library="zetex" deviceset="NPNSOT223" device=""/>
+<part name="T2" library="zetex" deviceset="NPNSOT223" device=""/>
+<part name="T3" library="zetex" deviceset="NPNSOT223" device=""/>
 </parts>
 <sheets>
@@
 <instance part="U$1" gate="G$1" x="0" y="-5.08"/>
 <instance part="Q1" gate="G$1" x="40.64" y="86.36"/>
-<instance part="Q3" gate="G$1" x="25.4" y="88.9"/>
 <instance part="R1" gate="G$1" x="0" y="81.28" rot="R90"/>
 <instance part="R2" gate="G$1" x="12.7" y="88.9"/>
@@
 <instance part="R5" gate="G$1" x="7.62" y="63.5" rot="R90"/>
 <instance part="Q2" gate="G$1" x="119.38" y="83.82"/>
-<instance part="Q4" gate="G$1" x="104.14" y="86.36"/>
 <instance part="R6" gate="G$1" x="78.74" y="78.74" rot="R90"/>
 <instance part="R7" gate="G$1" x="91.44" y="86.36"/>
@@
 <instance part="R10" gate="G$1" x="86.36" y="60.96" rot="R90"/>
 <instance part="Q5" gate="G$1" x="119.38" y="22.86"/>
-<instance part="Q6" gate="G$1" x="104.14" y="25.4"/>
 <instance part="R11" gate="G$1" x="78.74" y="17.78" rot="R90"/>
 <instance part="R12" gate="G$1" x="91.44" y="25.4"/>
@@
 <instance part="X2" gate="-8" x="-27.94" y="25.4"/>
 <instance part="C1" gate="G$1" x="-22.86" y="10.16"/>
+<instance part="T1" gate="A" x="25.4" y="88.9"/>
+<instance part="T2" gate="A" x="104.14" y="86.36"/>
+<instance part="T3" gate="A" x="104.14" y="25.4"/>
 </instances>
 <busses>
@@
 <net name="N$1" class="0">
 <segment>
-<pinref part="Q3" gate="G$1" pin="C"/>
 <wire x1="40.64" y1="93.98" x2="38.1" y2="93.98" width="0.1524" layer="91"/>
 <wire x1="38.1" y1="93.98" x2="27.94" y2="93.98" width="0.1524" layer="91"/>
 <wire x1="27.94" y1="93.98" x2="27.94" y2="101.6" width="0.1524" layer="91"/>
-<junction x="27.94" y="93.98"/>
 <pinref part="Q1" gate="G$1" pin="P-G"/>
 <junction x="38.1" y="93.98"/>
+<pinref part="T1" gate="A" pin="C1"/>
+<junction x="27.94" y="93.98"/>
 </segment>
 </net>
@@
 <segment>
 <pinref part="R2" gate="G$1" pin="2"/>
-<pinref part="Q3" gate="G$1" pin="B"/>
 <wire x1="17.78" y1="88.9" x2="22.86" y2="88.9" width="0.1524" layer="91"/>
+<pinref part="T1" gate="A" pin="B"/>
 </segment>
 </net>
@@
 </segment>
 <segment>
-<pinref part="Q3" gate="G$1" pin="E"/>
 <wire x1="27.94" y1="83.82" x2="27.94" y2="78.74" width="0.1524" layer="91"/>
 <label x="27.94" y="78.74" size="1.778" layer="95"/>
+<pinref part="T1" gate="A" pin="E"/>
 </segment>
 <segment>
@@
 </segment>
 <segment>
-<pinref part="Q4" gate="G$1" pin="E"/>
 <wire x1="106.68" y1="81.28" x2="106.68" y2="76.2" width="0.1524" layer="91"/>
 <label x="106.68" y="76.2" size="1.778" layer="95"/>
+<pinref part="T2" gate="A" pin="E"/>
 </segment>
 <segment>
@@
 </segment>
 <segment>
-<pinref part="Q6" gate="G$1" pin="E"/>
 <wire x1="106.68" y1="20.32" x2="106.68" y2="15.24" width="0.1524" layer="91"/>
 <label x="106.68" y="15.24" size="1.778" layer="95"/>
+<pinref part="T3" gate="A" pin="E"/>
 </segment>
 <segment>
@@
 <net name="N$2" class="0">
 <segment>
-<pinref part="Q4" gate="G$1" pin="C"/>
 <wire x1="119.38" y1="91.44" x2="116.84" y2="91.44" width="0.1524" layer="91"/>
 <wire x1="116.84" y1="91.44" x2="106.68" y2="91.44" width="0.1524" layer="91"/>
 <wire x1="106.68" y1="91.44" x2="106.68" y2="99.06" width="0.1524" layer="91"/>
-<junction x="106.68" y="91.44"/>
 <pinref part="Q2" gate="G$1" pin="P-G"/>
 <junction x="116.84" y="91.44"/>
+<pinref part="T2" gate="A" pin="C1"/>
+<junction x="106.68" y="91.44"/>
 </segment>
 </net>
@@
 <segment>
 <pinref part="R7" gate="G$1" pin="2"/>
-<pinref part="Q4" gate="G$1" pin="B"/>
 <wire x1="96.52" y1="86.36" x2="101.6" y2="86.36" width="0.1524" layer="91"/>
+<pinref part="T2" gate="A" pin="B"/>
 </segment>
 </net>
@@
 <net name="N$11" class="0">
 <segment>
-<pinref part="Q6" gate="G$1" pin="C"/>
 <wire x1="119.38" y1="30.48" x2="116.84" y2="30.48" width="0.1524" layer="91"/>
 <wire x1="116.84" y1="30.48" x2="106.68" y2="30.48" width="0.1524" layer="91"/>
 <wire x1="106.68" y1="30.48" x2="106.68" y2="38.1" width="0.1524" layer="91"/>
-<junction x="106.68" y="30.48"/>
 <pinref part="Q5" gate="G$1" pin="P-G"/>
 <junction x="116.84" y="30.48"/>
+<pinref part="T3" gate="A" pin="C1"/>
+<junction x="106.68" y="30.48"/>
 </segment>
 </net>
@@
 <segment>
 <pinref part="R12" gate="G$1" pin="2"/>
-<pinref part="Q6" gate="G$1" pin="B"/>
 <wire x1="96.52" y1="25.4" x2="101.6" y2="25.4" width="0.1524" layer="91"/>
-</segment>
-</net>
+<pinref part="T3" gate="A" pin="B"/>
+</segment>
+</net>
